Commit message: feat: 为fishbot仿真模型添加碰撞惯性属性并创建房间世界
- 新增通用惯性参数宏定义文件
- 为各部件添加碰撞几何体和惯性计算
- 创建房间模型配置和仿真世界文件

File: simulation_ws/src/fishbot_description/urdf/fishbot/actuator/caster.urdf.xacro (robot description, xacro)
@@ -1,4 +1,5 @@
 <?xml version='1.0'?>
 <robot xmlns:xacro = "http://www.ros.org/wiki/xacro">
+    <xacro:include filename="$(find fishbot_description)/urdf/fishbot/common_inertial.xacro" />
     <xacro:macro name="caster_xacro" params=" caster_name  xyz">
         <link name="${caster_name}_link">
@@ -16,4 +17,17 @@
             </material>
         </visual>
+        <collision>
+            <!--沿着自己几何中心的偏移和旋转-->
+            <origin xyz="0.0 0.0 0.0" rpy="0.0 0.0 0.0"/>
+            <!--几何形状-->
+            <geometry>
+                <sphere radius="0.016"/>
+            </geometry>
+            <!--材质颜色-->
+            <material name="yellow">
+                <color rgba="1.0 1.0 0.0 0.8"/>
+            </material>
+        </collision>
+            <xacro:sphere_inertia m="0.05" r="0.016"/>
         </link>
         <!--机器人关节，用于组合机器人的部件-->

File: simulation_ws/src/fishbot_description/urdf/fishbot/actuator/wheel.urdf.xacro (robot description, xacro)
@@ -1,4 +1,5 @@
 <?xml version='1.0'?>
 <robot xmlns:xacro = "http://www.ros.org/wiki/xacro">
+    <xacro:include filename="$(find fishbot_description)/urdf/fishbot/common_inertial.xacro" />
     <xacro:macro name="wheel_xacro" params=" wheel_name  xyz">
         <link name="${wheel_name}_link">
@@ -17,4 +18,18 @@
             </material>
         </visual>
+        <collision>
+            <!--沿着自己几何中心的偏移和旋转-->
+            <origin xyz="0.0 0.0 0.0" rpy="1.57079 0.0 0.0"/>
+            <!--几何形状-->
+            <geometry>
+                <!--圆柱体 radius 半径 0.10m 高度 length 0.12m-->
+                <cylinder radius="0.032" length="0.04"/>
+            </geometry>
+            <!--材质颜色-->
+            <material name="yellow">
+                <color rgba="1.0 1.0 0.0 0.8"/>
+            </material>
+        </collision>
+            <xacro:cylinder_inertia m="0.1" r="0.032" h="0.04"/>
         </link>
         <!--机器人关节，用于组合机器人的部件-->
@@ -38,4 +53,14 @@
                 </material>
             </visual>
+            <collision>
+                <origin xyz="0.0 0.0 0.0" rpy="0.0 0.0 0.0" />
+                <geometry>
+                    <sphere radius="0.019"/>
+                </geometry>
+                <material name="gray">
+                    <color rgba="0.5 0.5 0.5 1.0"/>
+                </material>
+            </collision>
+            <xacro:sphere_inertia m="0.05" r="0.019"/>
         </link>
         <joint name="${caster_name}_joint" type="fixed">

File: simulation_ws/src/fishbot_description/urdf/fishbot/base.urdf.xacro (robot description, xacro)
@@ -1,21 +1,44 @@
 <?xml version='1.0'?>
-<robot xmlns:xacro = "http://www.ros.org/wiki/xacro">
+<robot xmlns:xacro="http://www.ros.org/wiki/xacro">
+    <xacro:include filename="$(find fishbot_description)/urdf/fishbot/common_inertial.xacro" />
     <xacro:macro name="base_xacro" params="length radius">
+        <link name="base_footprint" />
         <link name="base_link">
-        <!--部件外观描述-->
-        <visual>
-            <!--沿着自己几何中心的偏移和旋转-->
-            <origin xyz="0.0 0.0 0.0" rpy="0.0 0.0 0.0"/>
-            <!--几何形状-->
-            <geometry>
-                <!--圆柱体 radius 半径 0.10m 高度 length 0.12m-->
-                <cylinder radius="${radius}" length="${length}"/>
-            </geometry>
-            <!--材质颜色-->
-            <material name="white">
-                <color rgba="1.0 1.0 1.0 0.5"/>
-            </material>
-        </visual>
+            <!--部件外观描述-->
+            <visual>
+                <!--沿着自己几何中心的偏移和旋转-->
+                <origin xyz="0.0 0.0 0.0" rpy="0.0 0.0 0.0" />
+                <!--几何形状-->
+                <geometry>
+                    <!--圆柱体
+                    radius 半径 0.10m 高度 length 0.12m-->
+                    <cylinder radius="${radius}" length="${length}" />
+                </geometry>
+                <!--材质颜色-->
+                <material name="white">
+                    <color rgba="1.0 1.0 1.0 0.5" />
+                </material>
+            </visual>
+            <collision>
+                <!--沿着自己几何中心的偏移和旋转-->
+                <origin xyz="0.0 0.0 0.0" rpy="0.0 0.0 0.0" />
+                <!--几何形状-->
+                <geometry>
+                    <!--圆柱体
+                    radius 半径 0.10m 高度 length 0.12m-->
+                    <cylinder radius="${radius}" length="${length}" />
+                </geometry>
+                <!--材质颜色-->
+                <material name="white">
+                    <color rgba="1.0 1.0 1.0 0.5" />
+                </material>
+            </collision>
+            <xacro:cylinder_inertia m="1.0" r="${radius}" h = "${length}"/>
         </link>
+        <joint name="joint_name" type="fixed">
+            <origin xyz="0.0 0.0 ${length/2.0+0.032-0.001}" rpy="0.0 0.0 0.0" />
+            <parent link="base_footprint" />
+            <child link="base_link" />
+        </joint>
     </xacro:macro>
 </robot>

File: simulation_ws/src/fishbot_description/urdf/fishbot/sensor/camera.urdf.xacro (robot description, xacro)
@@ -1,4 +1,5 @@
 <?xml version='1.0'?>
 <robot xmlns:xacro = "http://www.ros.org/wiki/xacro">
+    <xacro:include filename="$(find fishbot_description)/urdf/fishbot/common_inertial.xacro" />
     <xacro:macro name="camera_xacro" params="xyz">
         <!--机器人的IMU部件，惯性测量单元传感器-->
@@ -17,4 +18,17 @@
                 </material>
             </visual>
+            <collision>
+                <!--沿着自己几何中心的偏移和旋转-->
+                <origin xyz="0.0 0.0 0.0" rpy="0.0 0.0 0.0"/>
+                <!--几何形状-->
+                <geometry>
+                    <box size="0.02 0.10 0.02"/>
+                </geometry>
+                <!--材质颜色-->
+                <material name="red">
+                    <color rgba="0.8 0.2 0.2 1.0"/>
+                </material>
+            </collision>
+            <xacro:box_inertia m="0.05" w="0.02" h="0.10" d="0.02"/>
         </link>
         <!--机器人关节，用于组合机器人的部件-->

File: simulation_ws/src/fishbot_description/urdf/fishbot/sensor/imu.urdf.xacro (robot description, xacro)
@@ -1,4 +1,5 @@
 <?xml version='1.0'?>
 <robot xmlns:xacro = "http://www.ros.org/wiki/xacro">
+    <xacro:include filename="$(find fishbot_description)/urdf/fishbot/common_inertial.xacro" />
     <xacro:macro name="imu_xacro" params="xyz">
         <!--机器人的IMU部件，惯性测量单元传感器-->
@@ -17,4 +18,17 @@
                 </material>
             </visual>
+            <collision>
+                <!--沿着自己几何中心的偏移和旋转-->
+                <origin xyz="0.0 0.0 0.0" rpy="0.0 0.0 0.0"/>
+                <!--几何形状-->
+                <geometry>
+                    <box size="0.02 0.02 0.02"/>
+                </geometry>
+                <!--材质颜色-->
+                <material name="black">
+                    <color rgba="0.0 0.0 0.0 0.5"/>
+                </material>
+            </collision>
+            <xacro:box_inertia m="0.015" w="0.02" h="0.02" d="0.02"/>
         </link>
         <!--机器人关节，用于组合机器人的部件-->

File: simulation_ws/src/fishbot_description/urdf/fishbot/sensor/laser.urdf.xacro (robot description, xacro)
@@ -1,4 +1,5 @@
 <?xml version='1.0'?>
 <robot xmlns:xacro = "http://www.ros.org/wiki/xacro">
+    <xacro:include filename="$(find fishbot_description)/urdf/fishbot/common_inertial.xacro" />
     <xacro:macro name="laser_xacro" params="xyz">
         <!-- 雷达支撑杆-->
@@ -17,4 +18,17 @@
                 </material>
             </visual>
+            <collision>
+                <!--沿着自己几何中心的偏移和旋转-->
+                <origin xyz="0.0 0.0 0.0" rpy="0.0 0.0 0.0"/>
+                <!--几何形状-->
+                <geometry>
+                    <cylinder radius="0.01" length="0.10"/>
+                </geometry>
+                <!--材质颜色-->
+                <material name="green">
+                    <color rgba="0.2 0.8 0.2 1.0"/>
+                </material>
+            </collision>
+            <xacro:cylinder_inertia m="0.1" r="0.01" h="0.10"/>
         </link>
         <!--机器人的IMU部件，惯性测量单元传感器-->
@@ -33,4 +47,17 @@
                 </material>
             </visual>
+            <collision>
+                <!--沿着自己几何中心的偏移和旋转-->
+                <origin rpy="0.0 0.0 0.0" xyz="0.0 0.0 0.0"/>
+                <!--几何形状-->
+                <geometry>
+                    <cylinder radius="0.02" length="0.05"/>
+                </geometry>
+                <!--材质颜色-->
+                <material name="green">
+                    <color rgba="0.2 0.8 0.2 1.0"/>
+                </material>
+            </collision>
+            <xacro:cylinder_inertia m="0.15" r="0.02" h="0.05"/>
         </link>
         <!--机器人关节，用于组合机器人的部件-->

Commit message: feat: 添加鱼形机器人Gazebo插件和传感器配置

File: simulation_ws/src/fishbot_description/urdf/fishbot/actuator/caster.urdf.xacro (robot description, xacro)
@@ -37,4 +37,10 @@
             <origin xyz="${xyz}" rpy="0.0 0.0 0.0" />
         </joint>
+        <gazebo reference="${caster_name}_link">
+            <mu1 value="0.0"/>
+            <mu2 value="0.0"/>
+            <kp value="1000000000.0"/>
+            <kd value="1.0"/>
+        </gazebo>
     </xacro:macro>
 </robot>

File: simulation_ws/src/fishbot_description/urdf/fishbot/actuator/wheel.urdf.xacro (robot description, xacro)
@@ -69,4 +69,10 @@
             <origin xyz="${xyz}" rpy="0.0 0.0 0.0" />
         </joint>
+        <gazebo reference="${wheel_name}_link">
+            <mu1 value="20.0"/>
+            <mu2 value="20.0"/>
+            <kp value="1000000000.0"/>
+            <kd value="20.0"/>
+        </gazebo>
     </xacro:macro>
 </robot>

File: simulation_ws/src/fishbot_description/urdf/fishbot/fishbot.urdf.xacro (robot description, xacro)
@@ -10,4 +10,8 @@
     <xacro:include filename="$(find fishbot_description)/urdf/fishbot/actuator/wheel.urdf.xacro"/>
     <xacro:include filename="$(find fishbot_description)/urdf/fishbot/actuator/caster.urdf.xacro"/>
+    <!-- 插件部分 -->
+    <xacro:include filename="$(find fishbot_description)/urdf/fishbot/plugins/gazebo_control_plugin.xacro"/>
+    <xacro:include filename="$(find fishbot_description)/urdf/fishbot/plugins/gazebo_sensor_plugin.xacro"/>
+    <!-- 机器人部分 -->
     <xacro:base_xacro length="0.12" radius="0.10" />
     <xacro:imu_xacro xyz ="0.0 0.0 0.02" />
@@ -18,3 +22,4 @@
     <xacro:caster_xacro  caster_name="front_caster" xyz="0.08 0.0 -0.076" />
     <xacro:caster_xacro  caster_name="back_wheel"  xyz="-0.08 0.0 -0.076" />
+    <xacro:gazebo_control_plugin />
 </robot>

File: simulation_ws/src/fishbot_description/urdf/fishbot/sensor/laser.urdf.xacro (robot description, xacro)
@@ -72,4 +72,10 @@
             <origin xyz="${xyz}" rpy="0.0 0.0 0.0" />
         </joint>
+        <gazebo reference="laser_cylinder_link">
+            <material>Gazebo/Black</material>
+        </gazebo>
+        <gazebo reference="laser_link">
+            <material>Gazebo/Black</material>
+        </gazebo>
     </xacro:macro>
 </robot>
