Commit message: feat(camera): 添加相机光学连接的link和joint
新增camera_optical_link部件及对应的固定关节，用于匹配ROS相机的光学框架变换规范，确保后续传感器数据处理的坐标系一致性

File: simulation_ws/src/fishbot_description/urdf/fishbot/sensor/camera.urdf.xacro (robot description, xacro)
@@ -32,4 +32,7 @@
             <xacro:box_inertia m="0.05" w="0.02" h="0.10" d="0.02"/>
         </link>
+         <link name="camera_optical_link">
+            <!--部件外观描述-->
+        </link>
         <!--机器人关节，用于组合机器人的部件-->
         <joint name="camera_joint" type="fixed">
@@ -38,4 +41,9 @@
             <origin xyz="${xyz}" rpy="0.0 0.0 0.0" />
         </joint>
+        <joint name="camera_optical_joint" type="fixed">
+            <parent link="camera_link" />
+            <child link="camera_optical_link" />
+            <origin xyz="0.0 0.0 0.0" rpy="${-pi/2} 0.0 ${-pi/2}" />
+        </joint>
     </xacro:macro>
 </robot>
