Commit message: feat(fishbot_description): 升级机器人模型配置和启动文件
优化机器人URDF模型结构，修正惯性参数、材质颜色和关节配置
调整控制器参数和激光传感器更新频率
更新launch启动文件和RViz配置，修复路径和参数问题
添加Gazebo插件配置，优化仿真环境设置

File: nav2_ws/src/fishbot_description/urdf/fishbot/actuator/caster.urdf.xacro (robot description, xacro)
@@ -1,46 +1,39 @@
-<?xml version='1.0'?>
-<robot xmlns:xacro = "http://www.ros.org/wiki/xacro">
-    <xacro:include filename="$(find fishbot_description)/urdf/fishbot/common_inertial.xacro" />
-    <xacro:macro name="caster_xacro" params=" caster_name  xyz">
-        <link name="${caster_name}_link">
-        <!--部件外观描述-->
-        <visual>
-            <!--沿着自己几何中心的偏移和旋转-->
-            <origin xyz="0.0 0.0 0.0" rpy="0.0 0.0 0.0"/>
-            <!--几何形状-->
-            <geometry>
-                <sphere radius="0.016"/>
-            </geometry>
-            <!--材质颜色-->
-            <material name="yellow">
-                <color rgba="1.0 1.0 0.0 0.8"/>
-            </material>
-        </visual>
-        <collision>
-            <!--沿着自己几何中心的偏移和旋转-->
-            <origin xyz="0.0 0.0 0.0" rpy="0.0 0.0 0.0"/>
-            <!--几何形状-->
-            <geometry>
-                <sphere radius="0.016"/>
-            </geometry>
-            <!--材质颜色-->
-            <material name="yellow">
-                <color rgba="1.0 1.0 0.0 0.8"/>
-            </material>
-        </collision>
-            <xacro:sphere_inertia m="0.05" r="0.016"/>
+<?xml version="1.0"?>
+<robot xmlns:xacro="http://www.ros.org/wiki/xacro">
+   <xacro:include filename="$(find fishbot_description)/urdf/fishbot/common_inertia.xacro" />
+    <xacro:macro name="caster_xacro" params="caster_name xyz">
+        <link name="${caster_name}_caster_link">
+            <visual>
+                <origin xyz="0 0 0" rpy="0 0 0" />
+                <geometry>
+                    <sphere radius="0.016" />
+                </geometry>
+                <material name="black">
+                    <color rgba="0.0 0.0 0.0 0.8"/>
+                </material>
+            </visual>
+            <collision>
+                <origin xyz="0 0 0" rpy="0 0 0" />
+                <geometry>
+                    <sphere radius="0.016" />
+                </geometry>
+                <material name="black">
+                    <color rgba="0.0 0.0 0.0 0.8"/>
+                </material>
+            </collision>
+            <xacro:sphere_inertia m="0.01" r="0.016" />
         </link>
-        <!--机器人关节，用于组合机器人的部件-->
-        <joint name="${caster_name}_joint" type="fixed">
+        <gazebo reference="${caster_name}_caster_link">
+            <mu1 value="0.0" />
+            <mu2 value="0.0" />
+            <kp value="1000000000.0" />
+            <kd value="1.0" />
+        </gazebo>
+        <joint name="${caster_name}_caster_joint" type="fixed">
             <parent link="base_link" />
-            <child link="${caster_name}_link" />
-            <origin xyz="${xyz}" rpy="0.0 0.0 0.0" />
+            <child link="${caster_name}_caster_link" />
+            <origin xyz="${xyz}" />
+            <axis xyz="0 0 0" />
         </joint>
-        <gazebo reference="${caster_name}_link">
-            <mu1 value="0.0"/>
-            <mu2 value="0.0"/>
-            <kp value="1000000000.0"/>
-            <kd value="1.0"/>
-        </gazebo>
     </xacro:macro>
 </robot>

File: nav2_ws/src/fishbot_description/urdf/fishbot/actuator/wheel.urdf.xacro (robot description, xacro)
@@ -1,78 +1,39 @@
-<?xml version='1.0'?>
-<robot xmlns:xacro = "http://www.ros.org/wiki/xacro">
-    <xacro:include filename="$(find fishbot_description)/urdf/fishbot/common_inertial.xacro" />
-    <xacro:macro name="wheel_xacro" params=" wheel_name  xyz">
-        <link name="${wheel_name}_link">
-        <!--部件外观描述-->
-        <visual>
-            <!--沿着自己几何中心的偏移和旋转-->
-            <origin xyz="0.0 0.0 0.0" rpy="1.57079 0.0 0.0"/>
-            <!--几何形状-->
-            <geometry>
-                <!--圆柱体 radius 半径 0.10m 高度 length 0.12m-->
-                <cylinder radius="0.032" length="0.04"/>
-            </geometry>
-            <!--材质颜色-->
-            <material name="yellow">
-                <color rgba="1.0 1.0 0.0 0.8"/>
-            </material>
-        </visual>
-        <collision>
-            <!--沿着自己几何中心的偏移和旋转-->
-            <origin xyz="0.0 0.0 0.0" rpy="1.57079 0.0 0.0"/>
-            <!--几何形状-->
-            <geometry>
-                <!--圆柱体 radius 半径 0.10m 高度 length 0.12m-->
-                <cylinder radius="0.032" length="0.04"/>
-            </geometry>
-            <!--材质颜色-->
-            <material name="yellow">
-                <color rgba="1.0 1.0 0.0 0.8"/>
-            </material>
-        </collision>
-            <xacro:cylinder_inertia m="0.1" r="0.032" h="0.04"/>
-        </link>
-        <!--机器人关节，用于组合机器人的部件-->
-        <joint name="${wheel_name}_joint" type="continuous">
-            <parent link="base_link" />
-            <child link="${wheel_name}_link" />
-            <origin xyz="${xyz}" rpy="0.0 0.0 0.0" />
-            <axis xyz="0 1 0"/>
-        </joint>
-    </xacro:macro>
-    <!-- 万向轮（尸体自由度，固定球） -->
-    <xacro:macro name="caster_xacro" params="caster_name xyz">
-        <link name="${caster_name}_link">
+<?xml version="1.0"?>
+<robot xmlns:xacro="http://www.ros.org/wiki/xacro">
+   <xacro:include filename="$(find fishbot_description)/urdf/fishbot/common_inertia.xacro" />
+    <xacro:macro name="wheel_xacro" params="wheel_name xyz">
+        <link name="${wheel_name}_wheel_link">
             <visual>
-                <origin xyz="0.0 0.0 0.0" rpy="0.0 0.0 0.0" />
+                <origin xyz="0 0 0" rpy="1.57079 0 0" />
                 <geometry>
-                    <sphere radius="0.019"/>
+                    <cylinder length="0.04" radius="0.032" />
                 </geometry>
-                <material name="gray">
-                    <color rgba="0.5 0.5 0.5 1.0"/>
+                <material name="black">
+                    <color rgba="0.0 0.0 0.0 0.8"/>
                 </material>
             </visual>
             <collision>
-                <origin xyz="0.0 0.0 0.0" rpy="0.0 0.0 0.0" />
+                <origin xyz="0 0 0" rpy="1.57079 0 0" />
                 <geometry>
-                    <sphere radius="0.019"/>
+                    <cylinder length="0.04" radius="0.032" />
                 </geometry>
-                <material name="gray">
-                    <color rgba="0.5 0.5 0.5 1.0"/>
+                <material name="black">
+                    <color rgba="0.0 0.0 0.0 0.8"/>
                 </material>
             </collision>
-            <xacro:sphere_inertia m="0.05" r="0.019"/>
+            <xacro:cylinder_inertia m="0.1" h="0.04" r="0.032"/>
         </link>
-        <joint name="${caster_name}_joint" type="fixed">
+        <gazebo reference="${wheel_name}_wheel_link">
+            <mu1 value="20.0" />
+            <mu2 value="20.0" />
+            <kp value="1000000000.0" />
+            <kd value="1.0" />
+        </gazebo>
+        <joint name="${wheel_name}_wheel_joint" type="continuous">
             <parent link="base_link" />
-            <child link="${caster_name}_link" />
-            <origin xyz="${xyz}" rpy="0.0 0.0 0.0" />
+            <child link="${wheel_name}_wheel_link" />
+            <origin xyz="${xyz}" />
+            <axis xyz="0 1 0" />
         </joint>
-        <gazebo reference="${wheel_name}_link">
-            <mu1 value="20.0"/>
-            <mu2 value="20.0"/>
-            <kp value="1000000000.0"/>
-            <kd value="20.0"/>
-        </gazebo>
     </xacro:macro>
 </robot>

File: nav2_ws/src/fishbot_description/urdf/fishbot/base.urdf.xacro (robot description, xacro)
@@ -1,44 +1,33 @@
-<?xml version='1.0'?>
+<?xml version="1.0"?>
 <robot xmlns:xacro="http://www.ros.org/wiki/xacro">
-    <xacro:include filename="$(find fishbot_description)/urdf/fishbot/common_inertial.xacro" />
+   <xacro:include filename="$(find fishbot_description)/urdf/fishbot/common_inertia.xacro" />
     <xacro:macro name="base_xacro" params="length radius">
-        <link name="base_footprint" />
+     <link name="base_footprint" />
+        <joint name="base_joint" type="fixed">
+            <parent link="base_footprint" />
+            <child link="base_link" />
+            <origin xyz="0.0 0.0 ${length/2.0+0.032-0.001}" rpy="0 0 0" />
+        </joint>
         <link name="base_link">
-            <!--部件外观描述-->
             <visual>
-                <!--沿着自己几何中心的偏移和旋转-->
-                <origin xyz="0.0 0.0 0.0" rpy="0.0 0.0 0.0" />
-                <!--几何形状-->
+                <origin xyz="0 0 0.0" rpy="0 0 0" />
                 <geometry>
-                    <!--圆柱体
-                    radius 半径 0.10m 高度 length 0.12m-->
-                    <cylinder radius="${radius}" length="${length}" />
+                    <cylinder length="${length}" radius="${length}" />
                 </geometry>
-                <!--材质颜色-->
-                <material name="white">
-                    <color rgba="1.0 1.0 1.0 0.5" />
+                <material name="blue">
+                    <color rgba="0.1 0.1 1.0 0.5"/>
                 </material>
             </visual>
             <collision>
-                <!--沿着自己几何中心的偏移和旋转-->
-                <origin xyz="0.0 0.0 0.0" rpy="0.0 0.0 0.0" />
-                <!--几何形状-->
+                <origin xyz="0 0 0.0" rpy="0 0 0" />
                 <geometry>
-                    <!--圆柱体
-                    radius 半径 0.10m 高度 length 0.12m-->
-                    <cylinder radius="${radius}" length="${length}" />
+                    <cylinder length="${length}" radius="${length}" />
                 </geometry>
-                <!--材质颜色-->
-                <material name="white">
-                    <color rgba="1.0 1.0 1.0 0.5" />
+                <material name="blue">
+                    <color rgba="0.1 0.1 1.0 0.5"/>
                 </material>
             </collision>
-            <xacro:cylinder_inertia m="1.0" r="${radius}" h = "${length}"/>
+            <xacro:cylinder_inertia m="1.0" r="${radius}" h="${length}"/>
         </link>
-        <joint name="joint_name" type="fixed">
-            <origin xyz="0.0 0.0 ${length/2.0+0.032-0.001}" rpy="0.0 0.0 0.0" />
-            <parent link="base_footprint" />
-            <child link="base_link" />
-        </joint>
     </xacro:macro>
 </robot>

File: nav2_ws/src/fishbot_description/urdf/fishbot/fishbot.urdf.xacro (robot description, xacro)
@@ -1,32 +1,28 @@
-<?xml version='1.0'?>
-<robot xmlns:xacro = "http://www.ros.org/wiki/xacro" name="fishbot">
-    <!-- 基础部分 base_link-->
-    <xacro:include filename="$(find fishbot_description)/urdf/fishbot/base.urdf.xacro"/>
-    <!-- 传感器部分-->
-    <xacro:include filename="$(find fishbot_description)/urdf/fishbot/sensor/imu.urdf.xacro"/>
-    <xacro:include filename="$(find fishbot_description)/urdf/fishbot/sensor/camera.urdf.xacro"/>
-    <xacro:include filename="$(find fishbot_description)/urdf/fishbot/sensor/laser.urdf.xacro"/>
-    <!--执行器部分-->
-    <xacro:include filename="$(find fishbot_description)/urdf/fishbot/actuator/wheel.urdf.xacro"/>
-    <xacro:include filename="$(find fishbot_description)/urdf/fishbot/actuator/caster.urdf.xacro"/>
-    <!-- 插件部分 -->
-    <xacro:include filename="$(find fishbot_description)/urdf/fishbot/plugins/gazebo_control_plugin.xacro"/>
-    <xacro:include filename="$(find fishbot_description)/urdf/fishbot/plugins/gazebo_sensor_plugin.xacro"/>
-    <!-- 控制器部分 -->
-    <xacro:include filename="$(find fishbot_description)/urdf/fishbot/fishbot.ros2_control.xacro"/>
-    <!-- 机器人部分 -->
-    <xacro:base_xacro length="0.12" radius="0.10" />
-    <xacro:imu_xacro xyz ="0.0 0.0 0.02" />
-    <xacro:camera_xacro xyz ="0.10 0.0 0.075" />
-    <xacro:laser_xacro xyz ="0.0 0.0 0.10" />
-    <xacro:wheel_xacro  wheel_name="left_wheel" xyz="0 0.10 -0.06" />
-    <xacro:wheel_xacro  wheel_name="right_wheel" xyz="0 -0.10 -0.06" />
-    <xacro:caster_xacro  caster_name="front_caster" xyz="0.08 0.0 -0.076" />
-    <xacro:caster_xacro  caster_name="back_wheel"  xyz="-0.08 0.0 -0.076" />
-    <!-- 不要再启用：该插件直接在 Gazebo 里给轮关节设速度，会把轮子锁在 0 速，
-         与 ros2_control（effort / diff_drive 控制器）冲突。二选一，此处保留 ros2_control。 -->
+<?xml version="1.0"?>
+<robot xmlns:xacro="http://www.ros.org/wiki/xacro" name="fishbot">
+    <xacro:include filename="$(find fishbot_description)/urdf/fishbot/base.urdf.xacro" />
+    <!-- 传感器组件 -->
+    <xacro:include filename="$(find fishbot_description)/urdf/fishbot/sensor/imu.urdf.xacro" />
+    <xacro:include filename="$(find fishbot_description)/urdf/fishbot/sensor/laser.urdf.xacro" />
+    <xacro:include filename="$(find fishbot_description)/urdf/fishbot/sensor/camera.urdf.xacro" />
+     <!-- 执行器组件 -->
+    <xacro:include filename="$(find fishbot_description)/urdf/fishbot/actuator/wheel.urdf.xacro" />
+    <xacro:include filename="$(find fishbot_description)/urdf/fishbot/actuator/caster.urdf.xacro" />
+    <xacro:base_xacro length="0.12" radius="0.1" />
+    <!-- 传感器 -->
+    <xacro:imu_xacro xyz="0 0 0.02" />
+    <xacro:laser_xacro xyz="0 0 0.10" />
+    <xacro:camera_xacro xyz="0.10 0 0.075" />
+    <!-- 执行器主动轮+从动轮 -->
+    <xacro:wheel_xacro wheel_name="left" xyz="0 0.10 -0.06" />
+    <xacro:wheel_xacro wheel_name="right" xyz="0 -0.10 -0.06" />
+    <xacro:caster_xacro caster_name="front" xyz="0.08 0.0 -0.076" />
+    <xacro:caster_xacro caster_name="back" xyz="-0.08 0.0 -0.076" />
+    <!-- Gazebo 插件 -->
+    <xacro:include filename="$(find fishbot_description)/urdf/fishbot/plugins/gazebo_control_plugin.xacro" />
     <!-- <xacro:gazebo_control_plugin /> -->
+    <xacro:include filename="$(find fishbot_description)/urdf/fishbot/fishbot.ros2_control.xacro" />
+    <xacro:fishbot_ros2_control />
+    <xacro:include filename="$(find fishbot_description)/urdf/fishbot/plugins/gazebo_sensor_plugin.xacro" />
     <xacro:gazebo_sensor_plugin />
-    <!-- 控制器部分 -->
-    <xacro:fishbot_ros2_control />
 </robot>

File: nav2_ws/src/fishbot_description/urdf/fishbot/plugins/gazebo_sensor_plugin.xacro (robot description, xacro)
@@ -13,6 +13,6 @@
                 </plugin>
                 <always_on>true</always_on>
-                <visualize>true</visualize>
-                <update_rate>5</update_rate>
+                <visualize>false</visualize>
+                <update_rate>10</update_rate>
                 <pose>0 0 0 0 0 0</pose>
 								<!-- 激光传感器配置 -->

File: nav2_ws/src/fishbot_description/urdf/fishbot/sensor/camera.urdf.xacro (robot description, xacro)
@@ -1,48 +1,38 @@
-<?xml version='1.0'?>
-<robot xmlns:xacro = "http://www.ros.org/wiki/xacro">
-    <xacro:include filename="$(find fishbot_description)/urdf/fishbot/common_inertial.xacro" />
+<?xml version="1.0"?>
+<robot xmlns:xacro="http://www.ros.org/wiki/xacro">
+   <xacro:include filename="$(find fishbot_description)/urdf/fishbot/common_inertia.xacro" />
     <xacro:macro name="camera_xacro" params="xyz">
-        <!--机器人的IMU部件，惯性测量单元传感器-->
+        <!-- ============相机模块================ -->
         <link name="camera_link">
-            <!--部件外观描述-->
             <visual>
-                <!--沿着自己几何中心的偏移和旋转-->
-                <origin xyz="0.0 0.0 0.0" rpy="0.0 0.0 0.0"/>
-                <!--几何形状-->
+                <origin xyz="0 0 0.0" rpy="0 0 0" />
                 <geometry>
-                    <box size="0.02 0.10 0.02"/>
+                    <box size="0.02 0.10 0.02" />
                 </geometry>
-                <!--材质颜色-->
-                <material name="red">
-                    <color rgba="0.8 0.2 0.2 1.0"/>
+                <material name="black">
+                    <color rgba="0.0 0.0 0.0 0.8"/>
                 </material>
             </visual>
             <collision>
-                <!--沿着自己几何中心的偏移和旋转-->
-                <origin xyz="0.0 0.0 0.0" rpy="0.0 0.0 0.0"/>
-                <!--几何形状-->
+                <origin xyz="0 0 0.0" rpy="0 0 0" />
                 <geometry>
-                    <box size="0.02 0.10 0.02"/>
+                    <box size="0.02 0.10 0.02" />
                 </geometry>
-                <!--材质颜色-->
-                <material name="red">
-                    <color rgba="0.8 0.2 0.2 1.0"/>
+                <material name="black">
+                    <color rgba="0.0 0.0 0.0 0.8"/>
                 </material>
             </collision>
-            <xacro:box_inertia m="0.05" w="0.02" h="0.10" d="0.02"/>
+            <xacro:box_inertia m="0.01" w="0.02" h="0.10" d="0.02" />
         </link>
-         <link name="camera_optical_link">
-            <!--部件外观描述-->
-        </link>
-        <!--机器人关节，用于组合机器人的部件-->
+        <link name="camera_optical_link"></link>
+        <joint name="camera_optical_joint" type="fixed">
+            <parent link="camera_link" />
+            <child link="camera_optical_link" />
+            <origin xyz="0 0 0" rpy="${-pi/2} 0 ${-pi/2}" />
+        </joint>
         <joint name="camera_joint" type="fixed">
             <parent link="base_link" />
             <child link="camera_link" />
-            <origin xyz="${xyz}" rpy="0.0 0.0 0.0" />
-        </joint>
-        <joint name="camera_optical_joint" type="fixed">
-            <parent link="camera_link" />
-            <child link="camera_optical_link" />
-            <origin xyz="0.0 0.0 0.0" rpy="${-pi/2} 0.0 ${-pi/2}" />
+            <origin xyz="${xyz}" />
         </joint>
     </xacro:macro>

File: nav2_ws/src/fishbot_description/urdf/fishbot/sensor/imu.urdf.xacro (robot description, xacro)
@@ -1,40 +1,31 @@
-<?xml version='1.0'?>
-<robot xmlns:xacro = "http://www.ros.org/wiki/xacro">
-    <xacro:include filename="$(find fishbot_description)/urdf/fishbot/common_inertial.xacro" />
+<?xml version="1.0"?>
+<robot xmlns:xacro="http://www.ros.org/wiki/xacro">
+   <xacro:include filename="$(find fishbot_description)/urdf/fishbot/common_inertia.xacro" />
     <xacro:macro name="imu_xacro" params="xyz">
-        <!--机器人的IMU部件，惯性测量单元传感器-->
         <link name="imu_link">
-            <!--部件外观描述-->
             <visual>
-                <!--沿着自己几何中心的偏移和旋转-->
-                <origin xyz="0.0 0.0 0.0" rpy="0.0 0.0 0.0"/>
-                <!--几何形状-->
+                <origin xyz="0 0 00" rpy="0 0 0" />
                 <geometry>
-                    <box size="0.02 0.02 0.02"/>
+                    <box size="0.02 0.02 0.02" />
                 </geometry>
-                <!--材质颜色-->
                 <material name="black">
-                    <color rgba="0.0 0.0 0.0 0.5"/>
+                    <color rgba="0 0 0 0.8" />
                 </material>
             </visual>
             <collision>
-                <!--沿着自己几何中心的偏移和旋转-->
-                <origin xyz="0.0 0.0 0.0" rpy="0.0 0.0 0.0"/>
-                <!--几何形状-->
+                <origin xyz="0 0 00" rpy="0 0 0" />
                 <geometry>
-                    <box size="0.02 0.02 0.02"/>
+                    <box size="0.02 0.02 0.02" />
                 </geometry>
-                <!--材质颜色-->
                 <material name="black">
-                    <color rgba="0.0 0.0 0.0 0.5"/>
+                    <color rgba="0 0 0 0.8" />
                 </material>
             </collision>
-            <xacro:box_inertia m="0.015" w="0.02" h="0.02" d="0.02"/>
+            <xacro:box_inertia m="0.01" w="0.02" d="0.02" h="0.02"/>
         </link>
-        <!--机器人关节，用于组合机器人的部件-->
         <joint name="imu_joint" type="fixed">
             <parent link="base_link" />
             <child link="imu_link" />
-            <origin xyz="${xyz}" rpy="0.0 0.0 0.0" />
+            <origin xyz="${xyz}" />
         </joint>
     </xacro:macro>
