Commit message: feat(fishbot_description): 升级机器人模型配置和启动文件
优化机器人URDF模型结构，修正惯性参数、材质颜色和关节配置
调整控制器参数和激光传感器更新频率
更新launch启动文件和RViz配置，修复路径和参数问题
添加Gazebo插件配置，优化仿真环境设置

File: nav2_ws/src/fishbot_description/urdf/fishbot/sensor/laser.urdf.xacro (robot description, xacro)
@@ -1,75 +1,6 @@
-<?xml version='1.0'?>
-<robot xmlns:xacro = "http://www.ros.org/wiki/xacro">
-    <xacro:include filename="$(find fishbot_description)/urdf/fishbot/common_inertial.xacro" />
+<?xml version="1.0"?>
+<robot xmlns:xacro="http://www.ros.org/wiki/xacro">
+   <xacro:include filename="$(find fishbot_description)/urdf/fishbot/common_inertia.xacro" />
     <xacro:macro name="laser_xacro" params="xyz">
-        <!-- 雷达支撑杆-->
-        <link name="laser_cylinder_link">
-            <!--部件外观描述-->
-            <visual>
-                <!--沿着自己几何中心的偏移和旋转-->
-                <origin xyz="0.0 0.0 0.0" rpy="0.0 0.0 0.0"/>
-                <!--几何形状-->
-                <geometry>
-                    <cylinder radius="0.01" length="0.10"/>
-                </geometry>
-                <!--材质颜色-->
-                <material name="green">
-                    <color rgba="0.2 0.8 0.2 1.0"/>
-                </material>
-            </visual>
-            <collision>
-                <!--沿着自己几何中心的偏移和旋转-->
-                <origin xyz="0.0 0.0 0.0" rpy="0.0 0.0 0.0"/>
-                <!--几何形状-->
-                <geometry>
-                    <cylinder radius="0.01" length="0.10"/>
-                </geometry>
-                <!--材质颜色-->
-                <material name="green">
-                    <color rgba="0.2 0.8 0.2 1.0"/>
-                </material>
-            </collision>
-            <xacro:cylinder_inertia m="0.1" r="0.01" h="0.10"/>
-        </link>
-        <!--机器人的IMU部件，惯性测量单元传感器-->
-        <link name="laser_link">
-            <!--部件外观描述-->
-            <visual>
-                <!--沿着自己几何中心的偏移和旋转-->
-                <origin rpy="0.0 0.0 0.0" xyz="0.0 0.0 0.0"/>
-                <!--几何形状-->
-                <geometry>
-                    <cylinder radius="0.02" length="0.05"/>
-                </geometry>
-                <!--材质颜色-->
-                <material name="green">
-                    <color rgba="0.2 0.8 0.2 1.0"/>
-                </material>
-            </visual>
-            <collision>
-                <!--沿着自己几何中心的偏移和旋转-->
-                <origin rpy="0.0 0.0 0.0" xyz="0.0 0.0 0.0"/>
-                <!--几何形状-->
-                <geometry>
-                    <cylinder radius="0.02" length="0.05"/>
-                </geometry>
-                <!--材质颜色-->
-                <material name="green">
-                    <color rgba="0.2 0.8 0.2 1.0"/>
-                </material>
-            </collision>
-            <xacro:cylinder_inertia m="0.15" r="0.02" h="0.05"/>
-        </link>
-        <!--机器人关节，用于组合机器人的部件-->
-        <joint name="laser_joint" type="fixed">
-            <parent link="laser_cylinder_link" />
-            <child link="laser_link" />
-            <origin xyz="0.0 0.0 0.075" rpy="0.0 0.0 0.0" />
-        </joint>
-        <joint name="laser_cylinder_joint" type="fixed">
-            <parent link="base_link" />
-            <child link="laser_cylinder_link" />
-            <origin xyz="${xyz}" rpy="0.0 0.0 0.0" />
-        </joint>
         <gazebo reference="laser_cylinder_link">
             <material>Gazebo/Black</material>
@@ -78,4 +9,58 @@
             <material>Gazebo/Black</material>
         </gazebo>
+        <!-- ============雷达支撑杆================ -->
+        <link name="laser_cylinder_link">
+            <visual>
+                <origin xyz="0 0 0" rpy="0 0 0" />
+                <geometry>
+                    <cylinder length="0.10" radius="0.01" />
+                </geometry>
+                <material name="black">
+                    <color rgba="0.0 0.0 0.0 0.8" />
+                </material>
+            </visual>
+            <collision>
+                <origin xyz="0 0 0" rpy="0 0 0" />
+                <geometry>
+                    <cylinder length="0.10" radius="0.01" />
+                </geometry>
+                <material name="black">
+                    <color rgba="0.0 0.0 0.0 0.8" />
+                </material>
+            </collision>
+            <xacro:cylinder_inertia m="0.01" r="0.01" h="0.10" />
+        </link>
+        <joint name="laser_cylinder_joint" type="fixed">
+            <parent link="base_link" />
+            <child link="laser_cylinder_link" />
+            <origin xyz="${xyz}" />
+        </joint>
+        <!-- ============雷达================ -->
+        <link name="laser_link">
+            <visual>
+                <origin xyz="0 0 0" rpy="0 0 0" />
+                <geometry>
+                    <cylinder length="0.02" radius="0.02" />
+                </geometry>
+                <material name="black">
+                    <color rgba="0.0 0.0 0.0 0.8" />
+                </material>
+            </visual>
+            <collision>
+                <origin xyz="0 0 0" rpy="0 0 0" />
+                <geometry>
+                    <cylinder length="0.02" radius="0.02" />
+                </geometry>
+                <material name="black">
+                    <color rgba="0.0 0.0 0.0 0.8" />
+                </material>
+            </collision>
+            <xacro:cylinder_inertia m="0.03" r="0.02" h="0.02" />
+        </link>
+        <joint name="laser_joint" type="fixed">
+            <parent link="laser_cylinder_link" />
+            <child link="laser_link" />
+            <origin xyz="0 0 0.05" />
+        </joint>
     </xacro:macro>
 </robot>
